File: Block1.kicad_sch (KiCad schematic)
At the start: 6 parts, among them J1 USB_C_Receptacle_USB2.0_16P, U2 USBLC6-2SC6

Commit message: Usb and ^Power Block added
Parts:
- removed J1: USB_C_Receptacle_USB2.0_16P, Connector_USB:USB_C_Receptacle_GCT_USB4105-xx-A_16P_TopMnt_Horizontal, symbol Connector:USB_C_Receptacle_USB2.0_16P
- removed R1, R2: 5.1kΩ, Resistor_SMD:R_0603_1608Metric, symbol Device:R
- removed R3, R4: 33Ω, Resistor_SMD:R_0603_1608Metric, symbol Device:R
- removed U2: USBLC6-2SC6, Package_TO_SOT_SMD:SOT-23-6, symbol Power_Protection:USBLC6-2SC6
