File: Block1.kicad_sch (KiCad schematic)
At the start: 1 part, among them J3 Conn_02x10_Odd_Even

Commit message: Circuit Compleated
Parts:
- removed J3: Conn_02x10_Odd_Even, Connector_PinHeader_2.54mm:PinHeader_2x10_P2.54mm_Vertical, symbol Connector_Generic:Conn_02x10_Odd_Even

Commit message: ports added
Parts:
- added J3: Conn_02x10_Odd_Even, Connector_PinHeader_2.54mm:PinHeader_2x10_P2.54mm_Vertical, symbol Connector_Generic:Conn_02x10_Odd_Even
Connections:
- new net 3.3V: J3.2 (Pin_2)
- new net 3.3V / VTREF: J3.1 (Pin_1)
- new net GND: J3.10 (Pin_10), J3.12 (Pin_12), J3.14 (Pin_14), J3.16 (Pin_16), J3.18 (Pin_18), J3.20 (Pin_20), J3.4 (Pin_4), J3.6 (Pin_6), J3.8 (Pin_8)
- new net JTAG_RTCK: J3.11 (Pin_11)
- new net JTAG_TCK: J3.9 (Pin_9)
- new net JTAG_TDI: J3.5 (Pin_5)
- new net JTAG_TDO: J3.13 (Pin_13)
- new net JTAG_TMS: J3.7 (Pin_7)
- new net JTAG_TRST: J3.3 (Pin_3)
- new net NC: J3.17 (Pin_17), J3.19 (Pin_19)
- new net RESET_N: J3.15 (Pin_15)
