File: project_3.kicad_pcb (KiCad board)
At the start: 2 copper layers, 104.4 x 40 mm, 52 parts, among them J1 USB_C_Receptacle_USB2.0_16P, J10 Conn_01x04, J2 Conn_01x06, J3 Conn_02x10_Odd_Even, J4 Conn_02x20_Odd_Even, J5 GPIO_PORT1, J6 Conn_01x06, J7 Conn_01x06, J8 Conn_01x06, J9 Conn_02x10_Odd_Even, Q1 AO3401A, Q2 BC847, SW1 SW_Push, SW2 SW_Push, U1 LPC2148FBD64, U2 USBLC6-2SC6, U3 AP2112K-3.3, Y1 12MHz

Commit message: M change
Parts:
- moved U2 50.9 mm to (182.0, 102.0)
- moved U3 38.8 mm to (168.4, 113.6)
- moved C9 34.0 mm to (132.0, 121.3)
- moved C10 32.5 mm to (136.0, 121.3)
- moved Q1 31.9 mm to (168.4, 107.1)
- moved J10 31.8 mm to (133.0, 114.8), turned to 180 degrees
- moved C12 26.5 mm to (147.0, 122.0)
- moved C8 26.0 mm to (137.5, 99.7), turned to 0 degrees
- moved C16 24.5 mm to (151.5, 122.0)
- moved C7 24.0 mm to (142.0, 99.7), turned to 0 degrees
- moved C6 22.1 mm to (146.5, 99.7), turned to 0 degrees
- moved C4 19.8 mm to (151.2, 99.7), turned to 0 degrees
- moved R5 14.6 mm to (188.0, 100.5)
- moved R6 14.2 mm to (192.0, 100.5)
- moved R7 12.5 mm to (169.5, 101.5)
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Routing:
- net GND: track 389.1 -> 0.00 mm, vias 8 -> 0
- net +3.3V: track 182.0 -> 0.00 mm, vias 3 -> 0
- net /Block 10/NC: track 162.8 -> 0.00 mm
- net /RESET_N: track 100.8 -> 0.00 mm, vias 4 -> 0
- net /P0.23: track 87.1 -> 0.00 mm, vias 2 -> 0
- net /Block 10/3.3V: track 87.0 -> 0.00 mm
- net Net-(J1-D--PadA7): track 79.9 -> 0.00 mm, vias 4 -> 0
- net Net-(J1-D+-PadA6): track 79.4 -> 0.00 mm, vias 4 -> 0
- net /Block 10/3V3_A: track 78.5 -> 0.00 mm, vias 2 -> 0
- net /Block 10/+3.3V: track 77.9 -> 0.00 mm
- net /USB_DP: track 72.7 -> 0.00 mm, vias 4 -> 0
- net /+5V_PROTECTED: track 69.9 -> 0.00 mm, vias 4 -> 0
- net /ISP_P0_14: track 68.8 -> 0.00 mm, vias 4 -> 0
- net /Block 10/VREF: track 68.5 -> 0.00 mm, vias 1 -> 0
- net /Block 10/P1.30: track 67.9 -> 0.00 mm
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