File: Block10.kicad_sch (KiCad schematic)
At the start: 3 parts, among them J2 Conn_01x06

Commit message: ports added
Parts:
- removed J2: Conn_01x06, Connector_PinHeader_2.54mm:PinHeader_1x06_P2.54mm_Vertical, symbol Connector_Generic:Conn_01x06
- removed R10, R11: R, Resistor_SMD:R_0603_1608Metric, symbol Device:R
- added J4: Conn_02x20_Odd_Even, Connector_PinHeader_2.54mm:PinHeader_2x20_P2.54mm_Vertical, symbol Connector_Generic:Conn_02x20_Odd_Even
- added J5: GPIO_PORT1, Connector_PinHeader_2.54mm:PinHeader_2x20_P2.54mm_Vertical, symbol Connector_Generic:Conn_02x20_Odd_Even
Connections:
- new net +3.3V: J5.31 (Pin_31), J5.33 (Pin_33)
- new net 3.3V: J4.33 (Pin_33), J4.35 (Pin_35)
- new net GND: J4.34 (Pin_34), J4.36 (Pin_36), J4.37 (Pin_37), J4.38 (Pin_38), J5.32 (Pin_32), J5.34 (Pin_34)
- new net NC: J4.25 (Pin_25), J4.27 (Pin_27), J4.28 (Pin_28), J4.39 (Pin_39), J4.40 (Pin_40), J5.17 (Pin_17), J5.18 (Pin_18), J5.19 (Pin_19), J5.20 (Pin_20), J5.21 (Pin_21), J5.22 (Pin_22), J5.23 (Pin_23), J5.24 (Pin_24), J5.25 (Pin_25), J5.26 (Pin_26), J5.27 (Pin_27), J5.28 (Pin_28), J5.29 (Pin_29), J5.30 (Pin_30), J5.35 (Pin_35), J5.36 (Pin_36), J5.37 (Pin_37), J5.38 (Pin_38), J5.39 (Pin_39), J5.40 (Pin_40)
- new net P0.0: J4.1 (Pin_1)
- new net P0.1: J4.2 (Pin_2)
- new net P0.10: J4.11 (Pin_11)
- new net P0.11: J4.12 (Pin_12)
- new net P0.12: J4.13 (Pin_13)
- new net P0.13: J4.14 (Pin_14)
- new net P0.14: J4.15 (Pin_15)
- new net P0.15: J4.16 (Pin_16)
- new net P0.16: J4.17 (Pin_17)
- new net P0.17: J4.18 (Pin_18)
- new net P0.18: J4.19 (Pin_19)
- new net P0.19: J4.20 (Pin_20)
- new net P0.2: J4.3 (Pin_3)
- new net P0.20: J4.21 (Pin_21)
- new net P0.21: J4.22 (Pin_22)
- new net P0.22: J4.23 (Pin_23)
- new net P0.23: J4.24 (Pin_24)
- new net P0.25: J4.26 (Pin_26)
- new net P0.28: J4.29 (Pin_29)
- new net P0.29: J4.30 (Pin_30)
- new net P0.3: J4.4 (Pin_4)
- new net P0.30: J4.31 (Pin_31)
- new net P0.31: J4.32 (Pin_32)
- new net P0.4: J4.5 (Pin_5)
- new net P0.5: J4.6 (Pin_6)
- new net P0.6: J4.7 (Pin_7)
- new net P0.7: J4.8 (Pin_8)
- new net P0.8: J4.9 (Pin_9)
- new net P0.9: J4.10 (Pin_10)
- new net P1.16: J5.1 (Pin_1)
- new net P1.17: J5.2 (Pin_2)
- new net P1.18: J5.3 (Pin_3)
- new net P1.19: J5.4 (Pin_4)
- new net P1.20: J5.5 (Pin_5)
- new net P1.21: J5.6 (Pin_6)
- new net P1.22: J5.7 (Pin_7)
- new net P1.23: J5.8 (Pin_8)
- new net P1.24: J5.9 (Pin_9)
- new net P1.25: J5.10 (Pin_10)
- new net P1.26: J5.11 (Pin_11)
- new net P1.27: J5.12 (Pin_12)
- new net P1.28: J5.13 (Pin_13)
- new net P1.29: J5.14 (Pin_14)
- new net P1.30: J5.15 (Pin_15)
- new net P1.31: J5.16 (Pin_16)

Commit message: Circuit Compleated
Parts:
- added J10: Conn_01x04, Connector_PinHeader_2.54mm:PinHeader_1x04_P2.54mm_Vertical, symbol Connector_Generic:Conn_01x04
- added J2, J6, J7, J8: Conn_01x06, Connector_PinHeader_2.54mm:PinHeader_1x06_P2.54mm_Vertical, symbol Connector_Generic:Conn_01x06
- added J3, J9: Conn_02x10_Odd_Even, Connector_PinHeader_2.54mm:PinHeader_2x10_P2.54mm_Vertical, symbol Connector_Generic:Conn_02x10_Odd_Even
Connections:
- net +3.3V: now also J6.3 (Pin_3), J7.1 (Pin_1), J8.1 (Pin_1), J9.19 (Pin_19)
- net 3.3V: now also J2.1 (Pin_1), J3.2 (Pin_2)
- net GND: now also J10.4 (Pin_4), J2.2 (Pin_2), J3.10 (Pin_10), J3.12 (Pin_12), J3.14 (Pin_14), J3.16 (Pin_16), J3.18 (Pin_18), J3.20 (Pin_20), J3.4 (Pin_4), J3.6 (Pin_6), J3.8 (Pin_8), J6.2 (Pin_2), J6.4 (Pin_4), J7.2 (Pin_2), J8.2 (Pin_2), J9.17 (Pin_17), J9.18 (Pin_18)
- net NC: now also J3.17 (Pin_17), J3.19 (Pin_19), J9.20 (Pin_20)
- net P1.26 renamed JTAG_RTCK
- net JTAG_RTCK: now also J3.11 (Pin_11)
- net P1.27 renamed JTAG_TDO
- net JTAG_TDO: now also J3.13 (Pin_13)
- net P1.28 renamed JTAG_TDI
- net JTAG_TDI: now also J3.5 (Pin_5)
- net P1.29 renamed JTAG_TCK
- net JTAG_TCK: now also J3.9 (Pin_9)
- net P1.30 renamed JTAG_TMS
- net JTAG_TMS: now also J3.7 (Pin_7)
- net P1.31 renamed JTAG_TRST
- net JTAG_TRST: now also J3.3 (Pin_3)
- new net +5V_PROTECTED: J6.1 (Pin_1)
- new net 3.3V / VTREF: J3.1 (Pin_1)
- new net 3V3_A: J10.3 (Pin_3), J6.5 (Pin_5), J9.16 (Pin_16)
- new net AD0.1: J9.1 (Pin_1)
- new net AD0.2: J9.2 (Pin_2)
- new net AD0.3: J9.3 (Pin_3)
- new net AD0.4: J9.4 (Pin_4)
- new net AD0.6: J9.5 (Pin_5)
- new net AD0.7: J9.6 (Pin_6)
- new net AD1.0: J9.7 (Pin_7)
- new net AD1.1: J9.8 (Pin_8)
- new net AD1.2: J9.9 (Pin_9)
- new net AD1.3: J9.10 (Pin_10)
- new net AD1.4: J9.11 (Pin_11)
- new net AD1.5: J9.12 (Pin_12)
- new net AD1.6: J9.13 (Pin_13)
- new net AD1.7: J9.14 (Pin_14)
- new net AOUT: J10.1 (Pin_1)
- new net ISP_P0_14: J2.6 (Pin_6)
- new net MISO0: J7.4 (Pin_4)
- new net MOSI0: J7.5 (Pin_5)
- new net RESET_N: J2.5 (Pin_5), J3.15 (Pin_15)
- new net RXD0: J2.4 (Pin_4)
- new net SCK0: J7.3 (Pin_3)
- new net SCL0: J8.3 (Pin_3)
- new net SCL1: J8.5 (Pin_5)
- new net SDA0: J8.4 (Pin_4)
- new net SDA1: J8.6 (Pin_6)
- new net SSEL0: J7.6 (Pin_6)
- new net TXD0: J2.3 (Pin_3)
- new net VREF: J10.2 (Pin_2), J6.6 (Pin_6), J9.15 (Pin_15)
Other:
- company: (none) -> Devendra Kashyap
- moved on the sheet: J4, J5

Commit message: Upgraded
Other:
- moved on the sheet: J10, J2, J6
Changed lines of the file:
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@@
 	(wire
 		(pts
-			(xy 146.05 95.25) (xy 142.24 95.25)
+			(xy 196.85 93.98) (xy 200.66 93.98)
 		)
 		(stroke
@@
 	(wire
 		(pts
-			(xy 196.85 92.71) (xy 200.66 92.71)
+			(xy 196.85 109.22) (xy 200.66 109.22)
 		)
 		(stroke
@@
 	(wire
 		(pts
-			(xy 146.05 97.79) (xy 142.24 97.79)
+			(xy 196.85 96.52) (xy 200.66 96.52)
 		)
 		(stroke
@@
 	(wire
 		(pts
-			(xy 196.85 100.33) (xy 200.66 100.33)
+			(xy 196.85 116.84) (xy 200.66 116.84)
 		)
 		(stroke
@@
 	(wire
 		(pts
-			(xy 196.85 95.25) (xy 200.66 95.25)
+			(xy 196.85 111.76) (xy 200.66 111.76)
 		)
 		(stroke
@@
 	(wire
 		(pts
-			(xy 193.04 30.48) (xy 200.66 30.48)
+			(xy 193.04 31.75) (xy 200.66 31.75)
 		)
 		(stroke
@@
 	(wire
 		(pts
-			(xy 146.05 102.87) (xy 142.24 102.87)
+			(xy 196.85 101.6) (xy 200.66 101.6)
 		)
 		(stroke
@@
 	(wire
 		(pts
-			(xy 193.04 27.94) (xy 200.66 27.94)
+			(xy 193.04 29.21) (xy 200.66 29.21)
 		)
 		(stroke
@@
 	(wire
 		(pts
-			(xy 193.04 22.86) (xy 200.66 22.86)
+			(xy 193.04 24.13) (xy 200.66 24.13)
 		)
 		(stroke
@@
 	(wire
 		(pts
-			(xy 193.04 33.02) (xy 200.66 33.02)
+			(xy 193.04 34.29) (xy 200.66 34.29)
 		)
 		(stroke
@@
 	(wire
 		(pts
-			(xy 193.04 35.56) (xy 200.66 35.56)
+			(xy 193.04 36.83) (xy 200.66 36.83)
 		)
 		(stroke
@@
 	(wire
 		(pts
-			(xy 146.05 100.33) (xy 142.24 100.33)
+			(xy 196.85 99.06) (xy 200.66 99.06)
 		)
 		(stroke
@@
 	(wire
 		(pts
-			(xy 142.24 92.71) (xy 146.05 92.71)
+			(xy 200.66 91.44) (xy 196.85 91.44)
 		)
 		(stroke
@@
 	(wire
 		(pts
-			(xy 196.85 97.79) (xy 200.66 97.79)
+			(xy 196.85 114.3) (xy 200.66 114.3)
 		)
 		(stroke
@@
 	(wire
 		(pts
-			(xy 193.04 25.4) (xy 200.66 25.4)
+			(xy 193.04 26.67) (xy 200.66 26.67)
 		)
 		(stroke
@@
 	(wire
 		(pts
-			(xy 146.05 90.17) (xy 142.24 90.17)
+			(xy 196.85 88.9) (xy 200.66 88.9)
 		)
 		(stroke
@@
 	)
 	(label "GND"
-		(at 146.05 92.71 0)
+		(at 196.85 91.44 180)
 		(effects
 			(font
 				(size 1.27 1.27)
 			)
-			(justify left bottom)
+			(justify right bottom)
 		)
 	)
@@
 	)
 	(label "RXD0"
-		(at 146.05 97.79 0)
+		(at 196.85 96.52 180)
 		(effects
 			(font
 				(size 1.27 1.27)
 			)
-			(justify left bottom)
+			(justify right bottom)
 		)
 	)
@@
 	)
 	(label "+3.3V"
-		(at 193.04 27.94 180)
+		(at 193.04 29.21 180)
 		(effects
 			(font
@@
 	)
 	(label "GND"
-		(at 193.04 30.48 180)
+		(at 193.04 31.75 180)
 		(effects
 			(font
@@
 	)
 	(label "AOUT"
-		(at 196.85 92.71 180)
+		(at 196.85 109.22 180)
 		(effects
 			(font
@@
 	)
 	(label "TXD0"
-		(at 146.05 95.25 0)
+		(at 196.85 93.98 180)
 		(effects
 			(font
 				(size 1.27 1.27)
 			)
-			(justify left bottom)
+			(justify right bottom)
 		)
 	)
@@
 	)
 	(label "RESET_N"
-		(at 146.05 100.33 0)
+		(at 196.85 99.06 180)
 		(effects
 			(font
 				(size 1.27 1.27)
 			)
-			(justify left bottom)
+			(justify right bottom)
 		)
 	)
@@
 	)
 	(label "GND"
-		(at 193.04 25.4 180)
+		(at 193.04 26.67 180)
 		(effects
 			(font
@@
 	)
 	(label "+5V_PROTECTED"
-		(at 193.04 22.86 180)
+		(at 193.04 24.13 180)
 		(effects
 			(font
@@
 	)
 	(label "ISP_P0_14"
-		(at 146.05 102.87 0)
+		(at 196.85 101.6 180)
 		(effects
 			(font
 				(size 1.27 1.27)
 			)
-			(justify left bottom)
+			(justify right bottom)
 		)
 	)
@@
 	)
 	(label "3V3_A"
-		(at 193.04 33.02 180)
+		(at 193.04 34.29 180)
 		(effects
 			(font
@@
 	)
 	(label "3V3_A"
-		(at 196.85 97.79 180)
+		(at 196.85 114.3 180)
 		(effects
 			(font
@@
 	)
 	(label "3.3V"
-		(at 146.05 90.17 0)
+		(at 196.85 88.9 180)
 		(effects
 			(font
 				(size 1.27 1.27)
 			)
-			(justify left bottom)
+			(justify right bottom)
 		)
 	)
@@
 	)
 	(label "GND"
-		(at 196.85 100.33 180)
+		(at 196.85 116.84 180)
 		(effects
 			(font
@@
 	)
 	(label "VREF"
-		(at 193.04 35.56 180)
+		(at 193.04 36.83 180)
 		(effects
 			(font
@@
 	)
 	(label "VREF"
-		(at 196.85 95.25 180)
+		(at 196.85 111.76 180)
 		(effects
 			(font
@@
 	(symbol
 		(lib_id "Connector_Generic:Conn_01x04")
-		(at 205.74 95.25 0)
+		(at 205.74 111.76 0)
 		(unit 1)
 		(body_style 1)
@@
 		(fields_autoplaced yes)
 		(property "Reference" "J10"
-			(at 208.28 95.2499 0)
+			(at 208.28 111.7599 0)
 			(show_name no)
 			(do_not_autoplace no)
@@
 		)
 		(property "Value" "Conn_01x04"
-			(at 208.28 97.7899 0)
+			(at 208.28 114.2999 0)
 			(show_name no)
 			(do_not_autoplace no)
@@
 		)
 		(property "Footprint" "Connector_PinHeader_2.54mm:PinHeader_1x04_P2.54mm_Vertical"
-			(at 205.74 95.25 0)
+			(at 205.74 111.76 0)
 			(hide yes)
 			(show_name no)
@@
 		)
 		(property "Datasheet" ""
-			(at 205.74 95.25 0)
+			(at 205.74 111.76 0)
 			(hide yes)
 			(show_name no)
@@
 		)
 		(property "Description" "Generic connector, single row, 01x04, script generated (kicad-library-utils/schlib/autogen/connector/)"
-			(at 205.74 95.25 0)
+			(at 205.74 111.76 0)
 			(hide yes)
 			(show_name no)
@@
 	(symbol
 		(lib_id "Connector_Generic:Conn_01x06")
-		(at 137.16 95.25 0)
-		(mirror y)
+		(at 205.74 93.98 0)
 		(unit 1)
 		(body_style 1)
@@
 		(fields_autoplaced yes)
 		(property "Reference" "J2"
-			(at 134.62 95.2499 0)
+			(at 208.28 93.9799 0)
 			(show_name no)
 			(do_not_autoplace no)
@@
 		)
 		(property "Value" "Conn_01x06"
-			(at 134.62 97.7899 0)
+			(at 208.28 96.5199 0)
 			(show_name no)
 			(do_not_autoplace no)
@@
 		)
 		(property "Footprint" "Connector_PinHeader_2.54mm:PinHeader_1x06_P2.54mm_Vertical"
-			(at 137.16 95.25 0)
+			(at 205.74 93.98 0)
 			(hide yes)
 			(show_name no)
@@
 		)
 		(property "Datasheet" ""
-			(at 137.16 95.25 0)
+			(at 205.74 93.98 0)
 			(hide yes)
 			(show_name no)
@@
 		)
 		(property "Description" "Generic connector, single row, 01x06, script generated (kicad-library-utils/schlib/autogen/connector/)"
-			(at 137.16 95.25 0)
+			(at 205.74 93.98 0)
 			(hide yes)
 			(show_name no)
@@
 	(symbol
 		(lib_id "Connector_Generic:Conn_01x06")
-		(at 205.74 27.94 0)
+		(at 205.74 29.21 0)
 		(unit 1)
 		(body_style 1)
@@
 		(fields_autoplaced yes)
 		(property "Reference" "J6"
-			(at 208.28 27.9399 0)
+			(at 208.28 29.2099 0)
 			(show_name no)
 			(do_not_autoplace no)
@@
 		)
 		(property "Value" "Conn_01x06"
-			(at 208.28 30.4799 0)
+			(at 208.28 31.7499 0)
 			(show_name no)
 			(do_not_autoplace no)
@@
 		)
 		(property "Footprint" "Connector_PinHeader_2.54mm:PinHeader_1x06_P2.54mm_Vertical"
-			(at 205.74 27.94 0)
+			(at 205.74 29.21 0)
 			(hide yes)
 			(show_name no)
@@
 		)
 		(property "Datasheet" ""
-			(at 205.74 27.94 0)
+			(at 205.74 29.21 0)
 			(hide yes)
 			(show_name no)
@@
 		)
 		(property "Description" "Generic connector, single row, 01x06, script generated (kicad-library-utils/schlib/autogen/connector/)"
-			(at 205.74 27.94 0)
+			(at 205.74 29.21 0)
 			(hide yes)
 			(show_name no)
